File: gaia-primary.kicad_pcb (KiCad board)
At the start: 6 copper layers, 50 x 50 mm, 66 parts, among them IC2 ADXL375BCCZ, J1 Debug Connectors, J2 Conn_02x10_Odd_Even, J3 Conn_02x10_Odd_Even, Q1 BSS138, Q2 BSS138, U10 AP2112K-1.8, U11 AP2112K-3.3, U12 ICM-20948, U13 ICM-20948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

Commit message: routing to 6L + generating production files
Parts:
- moved Y1 0.10 mm to (175.9, 78.4)
Routing:
- net GND: track 86.3 -> 56.4 mm, vias 33 -> 104
- net /LOCAL_SDA: track 115.5 -> 95.7 mm, vias 3 -> 2
- net +3.3V: track 61.2 -> 45.1 mm, vias 16 -> 18
- net /DEBUG_USART_TX: track 62.5 -> 70.3 mm, vias 0 -> 1
- net /LOCAL_SCL: track 101.9 -> 96.0 mm, vias 3 -> 4
- net /DEBUG_NRST: track 58.5 -> 52.7 mm
- net /SPI1_SCK: track 86.1 -> 90.3 mm, vias 3 -> 4
- net /DEBUG_SWD_IO: track 50.3 -> 46.9 mm, vias 2 -> 1
- net /READY1: track 51.7 -> 48.8 mm
- net /SPI1_CS1: track 65.5 -> 67.0 mm, vias 2 -> 4
- net /DEBUG_SWD_CLK: track 42.9 -> 44.5 mm, vias 0 -> 1
- net /DEBUG_USART_RX: track 51.3 -> 50.7 mm, vias 2 -> 1
Other:
- board text added: "revision 1.1 Designed by Tamás Pécsi"
- board text removed: "revision 1.0 Designed by Tamás Pécsi"
